File: schematic/rx2.sch (KiCad schematic (older format))
At the start: 61 parts, among them J4 AudioJack3, Q11 2N3904, Q12 2N3904, Q13 2N7000, T2 FT37-43, U6 ADE-1, U7 L7809, U8 LM386, Y2 9 MHz, Y3 9 MHz, Y4 9 MHz, Y5 9 MHz, Y6 9 MHz

Commit message: Fix typo: 400u -> 470u
Parts:
- C78: value 400u -> 470u
Changed lines of the file:
@@
 P 9600 3100
 F 0 "C78" H 9715 3146 50  0000 L CNN
-F 1 "400u" H 9715 3055 50  0000 L CNN
+F 1 "470u" H 9715 3055 50  0000 L CNN
 F 2 "" H 9600 3100 50  0001 C CNN
 F 3 "~" H 9600 3100 50  0001 C CNN

Commit message: Some minor tweaks
Other:
- moved on the sheet: C70
Changed lines of the file:
@@
 	0    -1   -1   0
 $EndComp
-$Comp
-L Device:R R?
-U 1 1 62D7544D
-P 10150 2200
-AR Path="/62C0C022/62D7544D" Ref="R?"  Part="1"
-AR Path="/62CCEF11/62D7544D" Ref="R27"  Part="1"
-F 0 "R27" V 9943 2200 50  0000 C CNN
-F 1 "3.3K" V 10034 2200 50  0000 C CNN
-F 2 "" V 10080 2200 50  0001 C CNN
-F 3 "~" H 10150 2200 50  0001 C CNN
-	1    10150 2200
-	0    1    1    0
-$EndComp
-$Comp
-L Device:C C75
-U 1 1 62D7598D
-P 10400 2550
-F 0 "C75" H 10515 2596 50  0000 L CNN
-F 1 "47n" H 10515 2505 50  0000 L CNN
-F 2 "" H 10438 2400 50  0001 C CNN
-F 3 "~" H 10400 2550 50  0001 C CNN
-	1    10400 2550
-	1    0    0    -1
-$EndComp
-Text GLabel 10600 2200 2    50   Output ~ 0
+Text GLabel 10550 2200 2    50   Output ~ 0
 AFAMP_IN
-$Comp
-L power:GND #PWR?
-U 1 1 62D76BC9
-P 10400 2800
-AR Path="/62C0C022/62D76BC9" Ref="#PWR?"  Part="1"
-AR Path="/62CCEF11/62D76BC9" Ref="#PWR0104"  Part="1"
-F 0 "#PWR0104" H 10400 2550 50  0001 C CNN
-F 1 "GND" H 10405 2627 50  0001 C CNN
-F 2 "" H 10400 2800 50  0001 C CNN
-F 3 "" H 10400 2800 50  0001 C CNN
-	1    10400 2800
-	1    0    0    -1
-$EndComp
 Wire Wire Line
 	7650 2450 7750 2450
@@
 Wire Wire Line
 	9250 2200 9250 2100
-Wire Wire Line
-	9850 2200 10000 2200
-Wire Wire Line
-	10300 2200 10400 2200
-Wire Wire Line
-	10400 2200 10400 2400
-Connection ~ 10400 2200
-Wire Wire Line
-	10400 2200 10600 2200
-Wire Wire Line
-	10400 2700 10400 2800
 Wire Wire Line
 	9250 2950 9250 2800
@@
 Wire Wire Line
 	1800 5550 1800 5250
-Wire Wire Line
-	1800 5250 1600 5250
 $Comp
 L Amplifier_Audio:LM386 U8
@@
 Text Notes 2000 2600 0    50   ~ 0
 High-Q (>= 100 000) crystals are required to get\na narrowband CW filter with low losses. The crystals\nshould be measured using G3UUR method and\nmatched by the resonant frequency. Use LTspice\nto find the right capacitance for your crystals.
-Text GLabel 10600 1400 2    50   Output ~ 0
+Text GLabel 10650 1600 2    50   Output ~ 0
 S_METER_IN
 $Comp
 L Device:C C70
 U 1 1 6310FC29
-P 10400 1800
-F 0 "C70" H 10515 1846 50  0000 L CNN
-F 1 "22n" H 10515 1755 50  0000 L CNN
-F 2 "" H 10438 1650 50  0001 C CNN
-F 3 "~" H 10400 1800 50  0001 C CNN
-	1    10400 1800
-	1    0    0    -1
-$EndComp
-Wire Wire Line
-	10400 2200 10400 1950
-Wire Wire Line
-	10400 1650 10400 1400
-Wire Wire Line
-	10400 1400 10600 1400
+P 10350 1900
+F 0 "C70" H 10465 1946 50  0000 L CNN
+F 1 "22n" H 10465 1855 50  0000 L CNN
+F 2 "" H 10388 1750 50  0001 C CNN
+F 3 "~" H 10350 1900 50  0001 C CNN
+	1    10350 1900
+	1    0    0    -1
+$EndComp
+Wire Wire Line
+	10350 2200 10350 2050
+Wire Wire Line
+	10350 1750 10350 1600
+Wire Wire Line
+	10350 1600 10650 1600
+Wire Wire Line
+	1600 5250 1800 5250
+$Comp
+L Device:R R?
+U 1 1 62FE865F
+P 10100 2200
+AR Path="/62C0C022/62FE865F" Ref="R?"  Part="1"
+AR Path="/62CCEF11/62FE865F" Ref="R27"  Part="1"
+F 0 "R27" V 9893 2200 50  0000 C CNN
+F 1 "3.3K" V 9984 2200 50  0000 C CNN
+F 2 "" V 10030 2200 50  0001 C CNN
+F 3 "~" H 10100 2200 50  0001 C CNN
+	1    10100 2200
+	0    1    1    0
+$EndComp
+$Comp
+L Device:C C75
+U 1 1 62FE8669
+P 10350 2500
+F 0 "C75" H 10465 2546 50  0000 L CNN
+F 1 "47n" H 10465 2455 50  0000 L CNN
+F 2 "" H 10388 2350 50  0001 C CNN
+F 3 "~" H 10350 2500 50  0001 C CNN
+	1    10350 2500
+	1    0    0    -1
+$EndComp
+$Comp
+L power:GND #PWR?
+U 1 1 62FE8673
+P 10350 2800
+AR Path="/62C0C022/62FE8673" Ref="#PWR?"  Part="1"
+AR Path="/62CCEF11/62FE8673" Ref="#PWR0104"  Part="1"
+F 0 "#PWR0104" H 10350 2550 50  0001 C CNN
+F 1 "GND" H 10355 2627 50  0001 C CNN
+F 2 "" H 10350 2800 50  0001 C CNN
+F 3 "" H 10350 2800 50  0001 C CNN
+	1    10350 2800
+	1    0    0    -1
+$EndComp
+Wire Wire Line
+	10250 2200 10350 2200
+Wire Wire Line
+	10350 2200 10350 2350
+Connection ~ 10350 2200
+Wire Wire Line
+	10350 2650 10350 2800
+Wire Wire Line
+	9950 2200 9850 2200
+Wire Wire Line
+	10350 2200 10550 2200
 $EndSCHEMATC

Commit message: Correct the schematic
Parts:
- removed C75: 47n, symbol Device:C
- removed C86, C94: 10u, symbol Device:CP1
- removed R27: 3.3K, symbol Device:R
- added C74: 22u, symbol Device:CP1
- added RV1: 10K, symbol Device:R_POT_TRIM
- C88: renamed from C70; value 22n -> 2.2n
- U7: value L7809 -> L7805
- renumbered C71 to C70, C72 to C71, C73 to C72, C74 to C73, C76 to C75, C77 to C76, C78 to C77, C79 to C78, C80 to C79, C81 to C80, C82 to C81, C83 to C82, C84 to C83, C85 to C84, C87 to C85, C88 to C86, C89 to C87, C90 to C89, C91 to C90, C92 to C91, C93 to C92, C95 to C93, R28 to R27, R29 to R28, R30 to R29, R31 to R30, R32 to R31, R33 to R32, R34 to R33, R35 to R34, R36 to R35, R37 to R36, R38 to R37, R39 to R38, RV1 to RV2, RV2 to RV3
Connections:
- net AFAMP_IN: now also C88.1, C74.2; no longer C88.2
- net GND: now also RV1.1
- net S_METER_IN: now also C88.2; no longer C88.1
- net at C71.2: now also RV1.3
- net 9V_AUDIO renamed 5V_AUDIO
- new net: C74.1, RV1.2
- no-connect marks 0 -> 3
Other:
- note added: "Driver gain control"
- moved on the sheet: C85, C88
