File: schematic/s-meter.sch (KiCad schematic (older format))
At the start: 23 parts, among them Q24 2N3904, Q25 2N3904

Commit message: Fix typo: 400u -> 470u
Parts:
- C132, C133: value 400u -> 470u
Changed lines of the file:
@@
 AR Path="/63102909/6312A209" Ref="C132"  Part="1"
 F 0 "C132" H 4515 4696 50  0000 L CNN
-F 1 "400u" H 4515 4605 50  0000 L CNN
+F 1 "470u" H 4515 4605 50  0000 L CNN
 F 2 "" H 4400 4650 50  0001 C CNN
 F 3 "~" H 4400 4650 50  0001 C CNN
@@
 AR Path="/63102909/631478E5" Ref="C133"  Part="1"
 F 0 "C133" H 6215 4696 50  0000 L CNN
-F 1 "400u" H 6215 4605 50  0000 L CNN
+F 1 "470u" H 6215 4605 50  0000 L CNN
 F 2 "" H 6100 4650 50  0001 C CNN
 F 3 "~" H 6100 4650 50  0001 C CNN

Commit message: Some minor tweaks
Other:
- moved on the sheet: D23, R85
Changed lines of the file:
@@
 Comment4 ""
 $EndDescr
-Text GLabel 8350 3750 2    50   Output ~ 0
+Text GLabel 8500 3750 2    50   Output ~ 0
 S_METER_OUT
 Text GLabel 3200 4000 0    50   Input ~ 0
@@
 L Device:R R?
 U 1 1 63152289
-P 7750 4050
+P 7900 4050
 AR Path="/62C0C022/63152289" Ref="R?"  Part="1"
 AR Path="/62CCEF11/63152289" Ref="R?"  Part="1"
 AR Path="/63102909/63152289" Ref="R85"  Part="1"
-F 0 "R85" H 7820 4096 50  0000 L CNN
-F 1 "10K" H 7820 4005 50  0000 L CNN
-F 2 "" V 7680 4050 50  0001 C CNN
-F 3 "~" H 7750 4050 50  0001 C CNN
-	1    7750 4050
+F 0 "R85" H 7970 4096 50  0000 L CNN
+F 1 "10K" H 7970 4005 50  0000 L CNN
+F 2 "" V 7830 4050 50  0001 C CNN
+F 3 "~" H 7900 4050 50  0001 C CNN
+	1    7900 4050
 	1    0    0    -1
 $EndComp
@@
 L Device:LED D23
 U 1 1 63152BFF
-P 8100 4050
-F 0 "D23" V 8139 3932 50  0000 R CNN
-F 1 "Blue LED" V 8048 3932 50  0000 R CNN
-F 2 "" H 8100 4050 50  0001 C CNN
-F 3 "~" H 8100 4050 50  0001 C CNN
-	1    8100 4050
+P 8250 4050
+F 0 "D23" V 8289 3932 50  0000 R CNN
+F 1 "Blue LED" V 8198 3932 50  0000 R CNN
+F 2 "" H 8250 4050 50  0001 C CNN
+F 3 "~" H 8250 4050 50  0001 C CNN
+	1    8250 4050
 	0    -1   -1   0
 $EndComp
 Wire Wire Line
-	8350 3750 8100 3750
+	8500 3750 8250 3750
 Wire Wire Line
 	6350 3750 6700 3750
@@
 L power:GND #PWR?
 U 1 1 6315598B
-P 7750 4400
+P 7900 4400
 AR Path="/62C0C022/6315598B" Ref="#PWR?"  Part="1"
 AR Path="/62CCEF11/6315598B" Ref="#PWR?"  Part="1"
 AR Path="/63102909/6315598B" Ref="#PWR0187"  Part="1"
-F 0 "#PWR0187" H 7750 4150 50  0001 C CNN
-F 1 "GND" H 7755 4227 50  0001 C CNN
-F 2 "" H 7750 4400 50  0001 C CNN
-F 3 "" H 7750 4400 50  0001 C CNN
-	1    7750 4400
+F 0 "#PWR0187" H 7900 4150 50  0001 C CNN
+F 1 "GND" H 7905 4227 50  0001 C CNN
+F 2 "" H 7900 4400 50  0001 C CNN
+F 3 "" H 7900 4400 50  0001 C CNN
+	1    7900 4400
 	1    0    0    -1
 $EndComp
@@
 L power:GND #PWR?
 U 1 1 63155C32
-P 8100 4400
+P 8250 4400
 AR Path="/62C0C022/63155C32" Ref="#PWR?"  Part="1"
 AR Path="/62CCEF11/63155C32" Ref="#PWR?"  Part="1"
 AR Path="/63102909/63155C32" Ref="#PWR0188"  Part="1"
-F 0 "#PWR0188" H 8100 4150 50  0001 C CNN
-F 1 "GND" H 8105 4227 50  0001 C CNN
-F 2 "" H 8100 4400 50  0001 C CNN
-F 3 "" H 8100 4400 50  0001 C CNN
-	1    8100 4400
+F 0 "#PWR0188" H 8250 4150 50  0001 C CNN
+F 1 "GND" H 8255 4227 50  0001 C CNN
+F 2 "" H 8250 4400 50  0001 C CNN
+F 3 "" H 8250 4400 50  0001 C CNN
+	1    8250 4400
 	1    0    0    -1
 $EndComp
@@
 Wire Wire Line
 	7400 3750 7400 3900
+Wire Wire Line
+	7400 3750 7150 3750
+Wire Wire Line
+	7400 4200 7400 4400
+Wire Wire Line
+	7900 3750 7900 3900
+Connection ~ 7900 3750
+Wire Wire Line
+	7900 4200 7900 4400
+Wire Wire Line
+	8250 3750 8250 3900
+Connection ~ 8250 3750
+Wire Wire Line
+	8250 3750 7900 3750
+Wire Wire Line
+	8250 4200 8250 4400
+Text Notes 8400 4400 0    50   ~ 0
+The blue LED ensures the voltage\nwill not exceed 3V.
+Wire Wire Line
+	7400 3750 7900 3750
 Connection ~ 7400 3750
-Wire Wire Line
-	7400 3750 7150 3750
-Wire Wire Line
-	7400 4200 7400 4400
-Wire Wire Line
-	7750 3750 7750 3900
-Connection ~ 7750 3750
-Wire Wire Line
-	7750 3750 7400 3750
-Wire Wire Line
-	7750 4200 7750 4400
-Wire Wire Line
-	8100 3750 8100 3900
-Connection ~ 8100 3750
-Wire Wire Line
-	8100 3750 7750 3750
-Wire Wire Line
-	8100 4200 8100 4400
-Text Notes 8250 4400 0    50   ~ 0
-The blue LED ensures the voltage\nwill not exceed 3V.
 $EndSCHEMATC

Commit message: Correct the schematic
Parts:
- renumbered C127 to C125, C128 to C126, C129 to C127, C130 to C128, C131 to C129, C132 to C130, C133 to C131, R79 to R77, R80 to R78, R81 to R79, R82 to R80, R83 to R81, R84 to R82, R85 to R83, R86 to R84, R87 to R85, R88 to R86, R89 to R87
